File: Quad_ESC.brd (EAGLE design)
At the start: 96.5 x 40.1 mm, 28 parts, among them Y1 ECS-80-S-4X

Commit message: Quick, Minor Changes
Parts:
- moved U$10 0.13 mm to (13.3, 6.60)
Routing:
- net +12V: track 129.6 -> 139.0 mm
- net +3V3: track 140.9 -> 141.8 mm
- net TLM: track 56.5 -> 57.1 mm
- net NRST1: track 12.0 -> 12.6 mm
